File: hardware/EcoNode-Sentinel.kicad_pcb (KiCad board)
At the start: 4 copper layers, 0 parts

Commit message: hardware: configure 4-layer stackup matrix, power net classes, and floorplan day 4
Parts:
- added C1: 10uF, Capacitor_SMD:C_0805_2012Metric, F.Cu at (89.7, 105.1)
- added C2: 0.1uF, Capacitor_SMD:C_0603_1608Metric, F.Cu at (89.7, 109.6)
- added C3: 10uF, Capacitor_SMD:C_0805_2012Metric, F.Cu at (99.2, 105.1)
- added C4: 0.1uF, Capacitor_SMD:C_0603_1608Metric, F.Cu at (99.2, 109.6)
- added C5: 22uF, Capacitor_SMD:C_1206_3216Metric, F.Cu at (121.8, 89.6)
- added C6: 1uF, Capacitor_SMD:C_0603_1608Metric, F.Cu at (122.0, 93.6)
- added C7: 0.1uF, Capacitor_SMD:C_0603_1608Metric, F.Cu at (122.0, 97.1)
- added J1: USB_C_Receptacle_USB2.0_16P, Connector_USB:USB_C_Receptacle_GCT_USB4105-xx-A_16P_TopMnt_Horizontal, F.Cu at (77.7, 111.1)
- added R1: 5.1k, Resistor_SMD:R_0603_1608Metric, F.Cu at (75.4, 104.1)
- added R2: 5.1k, Resistor_SMD:R_0603_1608Metric, F.Cu at (80.2, 104.1)
- added U1: AP2112K-3.3, Package_TO_SOT_SMD:SOT-23-5, F.Cu at (94.2, 106.1)
- added U2: ESP32-S3-WROOM-1, RF_Module:ESP32-S3-WROOM-1, F.Cu at (119.7, 108.2)
